File: keyboard.kicad_pcb (KiCad board)
At the start: 2 copper layers, 3.7 x 3.7 mm, 319 parts, among them J1 USB-C, J2 ISP Header, J3 LED Extension, K1 ESC, K10 F9, K11 F10, K12 F11, K13 F12, K14 BCKTCK, K15 1, K16 2, K17 3, K18 4, K19 5, K2 F1, K20 6, K21 7, K22 8, K23 9, K24 0, K25 MINUS, K26 EQU, K27 BCKSPC, K28 PRNT, K29 SCRL, K3 F2, K30 PAUSE, K31 TAB, K32 Q, K33 W, K34 E, K35 R, K36 T, K37 Y, K38 U, K39 I, K4 F3, K40 O, K41 P, K42 OP_SQ, K43 CL_SQ, K44 ENTER, K45 INS, K46 HOME, K47 PG_UP, K48 CAPS, K49 A, K5 F4, K50 S, K51 D, K52 F, K53 G, K54 H, K55 J, K56 K, K57 L, K58 SEMICLN, K59 APOS, K6 F5, K60 HASH, K61 DEL, K62 END, K63 PG_DN, K64 L_SHIFT, K65 B_SLSH, K66 Z, K67 X, K68 C, K69 V, K7 F6, K70 B, K71 N, K72 M, K73 COMMA, K74 DOT, K75 F_SLSH, K76 R_SHIFT, K77 U_ARR, K78 L_CTRL, K79 L_WIN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

Commit message: more layout
Parts:
- D10, D100, D101, D102, D103, D104, D105, D106, D107, D108, D109, D11, D110, D111, D112, D113, D114, D115, D116, D117, D118, D119, D12, D120, D121, D122, D123, D124, D125, D126, D127, D128, D129, D13, D130, D131, D132, D133, D134, D135, D136, D137, D138, D139, D14, D140, D141, D142, D143, D144, D145, D146, D147, D148, D149, D15, D150, D151, D152, D153, D154, D155, D156, D157, D158, D159, D16, D160, D161, D162, D163, D164, D165, D166, D167, D168, D169, D17, D170, D171, D172, D173, D174, D175, D176, D177, D178, D179, D18, D180, D181, D19, D2, D20, D21, D22, D23, D24, D25, D26, D27, D3, D32, D33, D34, D35, D36, D37, D38, D39, D4, D40, D41, D42, D43, D44, D45, D46, D47, D48, D49, D5, D50, D51, D52, D53, D54, D55, D56, D57, D58, D59, D6, D60, D61, D62, D63, D64, D65, D66, D67, D68, D69, D7, D70, D71, D72, D73, D74, D75, D76, D77, D78, D79, D8, D80, D81, D82, D83, D84, D85, D86, D87, D88, D89, D9, D91, D92, D93, D94, D95, D96, D97, D98, D99, J3, R10: moved to B.Cu
- moved D15 488.6 mm to (49.4, 114.0), turned to 180 degrees
- moved D4 485.4 mm to (106.5, 85.4), turned to 180 degrees
- moved D34 484.2 mm to (97.0, 133.0), turned to 180 degrees
- moved D18 471.8 mm to (106.5, 114.0), turned to 180 degrees
- moved D16 468.5 mm to (68.4, 114.0), turned to 180 degrees
- moved D2 461.5 mm to (49.4, 85.4), turned to 180 degrees
- moved D3 461.5 mm to (87.5, 85.4), turned to 180 degrees
- moved D70 460.6 mm to (149.4, 171.1), turned to 180 degrees
- moved D49 456.3 mm to (56.5, 152.1), turned to 180 degrees
- moved D35 451.6 mm to (116.0, 133.0), turned to 180 degrees
- moved D79 444.3 mm to (51.7, 190.2), turned to 180 degrees
- moved D81 441.9 mm to (99.4, 190.2), turned to 180 degrees
- moved D33 441.7 mm to (77.9, 133.0), turned to 180 degrees
- moved D19 440.2 mm to (125.6, 114.0), turned to 180 degrees
- moved D22 418.4 mm to (182.7, 114.0), turned to 180 degrees
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- renumbered J2 to J1, J1 to J2, R7 to R5, R5 to R6, R8 to R7, R6 to R8
Connections:
- net Net-(C6-Pad1) renamed /MCU/XTAL1
- net Net-(C7-Pad1) renamed /MCU/XTAL2
- net Net-(C8-Pad1) renamed /MCU/UCAP
- net Net-(J1-PadA4) renamed /MCU/VBUS
- net Net-(J1-PadA5) renamed /MCU/CC1
- net Net-(J1-PadB5) renamed /MCU/CC2
- net Net-(R7-Pad1) renamed /MCU/MCU_D+
- net Net-(R8-Pad2) renamed /MCU/MCU_D-
- net Net-(R9-Pad1) renamed /MCU/~{HWB}
- J2 pad A6: Net-(J1-PadA6) -> /MCU/CON_D+
- J2 pad A7: Net-(J1-PadA7) -> /MCU/CON_D-
- J2 pad B6: Net-(J1-PadA6) -> /MCU/CON_D+
- J2 pad B7: Net-(J1-PadA7) -> /MCU/CON_D-
- R5 pad 2: Net-(J1-PadA7) -> /MCU/CON_D+
- R7 pad 1: Net-(J1-PadA6) -> /MCU/CON_D-
Routing:
- added copper zone on B.Cu, net GND
Other:
- board size 3.7 x 3.7 mm -> 348.6 x 131.8 mm

Commit message: rough layout complete
Parts:
- removed the TP1 at (389.9, 156.5)
- removed TP10, TP11, TP13, TP14, TP15, TP16, TP17: TestPoint, TestPoint:TestPoint_THTPad_D1.0mm_Drill0.5mm
- removed the TP2 at (399.0, 156.5)
- removed the TP3 at (402.1, 159.5)
- removed the TP4 at (389.9, 159.5)
- removed the TP5 at (399.0, 159.5)
- removed the TP6 at (399.0, 162.6)
- removed the TP7 at (392.9, 156.5)
- removed the TP8 at (396.0, 162.6)
- removed the TP9 at (402.1, 165.6)
- C1, C2, C3, C4, C6, C7: footprint Capacitor_SMD:C_0805_2012Metric_Pad1.18x1.45mm_HandSolder -> Capacitor_SMD:C_0402_1005Metric_Pad0.74x0.62mm_HandSolder; moved to B.Cu
- C5, C8: footprint Capacitor_SMD:C_0805_2012Metric_Pad1.18x1.45mm_HandSolder -> Capacitor_SMD:C_0603_1608Metric_Pad1.08x0.95mm_HandSolder; moved to B.Cu
- D1, D28, D29, D30, D31, J1, J2, SW1, TH1: moved to B.Cu
- R1, R2, R3, R4, R5, R8, R9: footprint Resistor_SMD:R_0805_2012Metric_Pad1.20x1.40mm_HandSolder -> Resistor_SMD:R_0603_1608Metric_Pad0.98x0.95mm_HandSolder; moved to B.Cu
- R10: footprint Resistor_SMD:R_0805_2012Metric_Pad1.20x1.40mm_HandSolder -> Resistor_SMD:R_0603_1608Metric_Pad0.98x0.95mm_HandSolder
- R6: renamed from R7; footprint Resistor_SMD:R_0805_2012Metric_Pad1.20x1.40mm_HandSolder -> Resistor_SMD:R_0603_1608Metric_Pad0.98x0.95mm_HandSolder; moved to B.Cu
- R7: renamed from R6; footprint Resistor_SMD:R_0805_2012Metric_Pad1.20x1.40mm_HandSolder -> Resistor_SMD:R_0603_1608Metric_Pad0.98x0.95mm_HandSolder; moved to B.Cu
- TP1: renamed from TP12; moved to B.Cu
- TP2: renamed from TP18; moved to B.Cu
- TP3: renamed from TP19; moved to B.Cu
- TP4: renamed from TP20; moved to B.Cu
- TP5: renamed from TP21; moved to B.Cu
- TP6: renamed from TP22; moved to B.Cu
- TP7: renamed from TP23; moved to B.Cu
- TP8: renamed from TP24; moved to B.Cu
- TP9: renamed from TP25; moved to B.Cu
- moved R7 150.8 mm to (317.8, 81.7)
- moved R8 145.4 mm to (323.0, 82.7), turned to -90 degrees
- moved TP8 140.2 mm to (324.4, 89.6), turned to 180 degrees
- moved TP9 139.1 mm to (324.5, 93.2), turned to 180 degrees
- moved TH1 136.5 mm to (325.1, 83.5), turned to 90 degrees
- moved R6 114.9 mm to (320.7, 153.9), turned to -90 degrees
- moved C1 113.9 mm to (315.9, 164.9), turned to -90 degrees
- moved TP2 110.2 mm to (317.7, 88.1), turned to 180 degrees
- moved C4 104.0 mm to (315.8, 172.1), turned to 90 degrees
- moved C2 103.3 mm to (331.2, 166.5), turned to -90 degrees
- moved C8 97.9 mm to (323.7, 159.8), turned to 90 degrees
- moved R9 97.2 mm to (318.2, 176.1), turned to 180 degrees
- moved C3 96.6 mm to (327.4, 175.9)
- moved R1 96.6 mm to (334.1, 164.9), turned to 90 degrees
- moved R3 96.6 mm to (334.7, 159.2)
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Routing:
- added copper zone on F.Cu, net GND
- removed copper zone on B.Cu, net GND

Commit message: before i fuck up
Parts:
- removed TP2, TP3, TP4, TP5, TP6, TP7: TestPoint, TestPoint:TestPoint_THTPad_D1.0mm_Drill0.5mm
- C1, C2, C3, C4, C6, C7: footprint Capacitor_SMD:C_0402_1005Metric_Pad0.74x0.62mm_HandSolder -> Capacitor_SMD:C_0603_1608Metric_Pad1.08x0.95mm_HandSolder
- moved TP9 15.0 mm to (314.8, 81.7)
- moved J3 11.4 mm to (371.1, 172.1)
- moved D64 7.83 mm to (370.2, 132.1), turned to 0 degrees
- moved R4 3.91 mm to (338.7, 157.8)
- moved R2 3.91 mm to (338.7, 156.2)
- moved R3 3.91 mm to (338.6, 159.4)
- moved SW1 3.46 mm to (344.7, 155.2)
- moved R7 3.23 mm to (320.0, 84.0), turned to 90 degrees
- moved TP8 2.53 mm to (325.1, 87.2)
- moved C3 1.55 mm to (327.5, 177.4)
- moved D1 1.45 mm to (337.8, 163.9)
- moved R1 1.45 mm to (335.5, 164.6)
- moved C7 1.36 mm to (335.4, 168.7)
- moved C6 1.34 mm to (335.4, 172.1)
- moved R8 1.32 mm to (322.9, 84.0)
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Routing:
- net /Key Matrix/ROW_2: track 0.00 -> 321.1 mm
- net /Key Matrix/ROW_1: track 0.00 -> 315.7 mm
- net /Key Matrix/ROW_0: track 0.00 -> 282.1 mm
- net /Key Matrix/ROW_3: track 0.00 -> 250.2 mm
- net /Key Matrix/COL_6: track 0.00 -> 121.1 mm
- net /Key Matrix/COL_2: track 0.00 -> 119.9 mm
- net /Key Matrix/COL_12: track 0.00 -> 119.8 mm
- net /Key Matrix/COL_11: track 0.00 -> 117.8 mm
- net /Key Matrix/COL_13: track 0.00 -> 112.4 mm
- net /Key Matrix/COL_0: track 0.00 -> 112.4 mm
- net /Key Matrix/COL_15: track 0.00 -> 107.4 mm
- net /Key Matrix/COL_16: track 0.00 -> 106.9 mm
- net /Key Matrix/COL_9: track 0.00 -> 101.7 mm
- net /Key Matrix/COL_8: track 0.00 -> 101.7 mm
- net /Key Matrix/COL_7: track 0.00 -> 100.8 mm
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- removed copper zone on F.Cu, net GND

Commit message: fucking with pinout
Parts:
- moved D14 13.1 mm to (302.9, 85.4), turned to 0 degrees
- moved D31 13.1 mm to (364.9, 85.4), turned to 0 degrees
- moved D48 13.1 mm to (364.9, 114.0), turned to 0 degrees
- moved D89 13.0 mm to (365.0, 190.2), turned to 0 degrees
- moved TP8 12.2 mm to (336.2, 82.1)
- moved R10 7.03 mm to (379.7, 102.2), turned to -90 degrees
- moved TP1 6.25 mm to (379.7, 105.0)
- moved D64 5.38 mm to (364.9, 133.0)
- moved D173 4.76 mm to (185.7, 195.3), turned to 0 degrees
- moved R7 4.56 mm to (317.7, 88.0)
- moved R8 4.56 mm to (325.2, 88.0)
- moved TH1 3.99 mm to (328.8, 82.2), turned to 180 degrees
- moved D170 2.38 mm to (126.2, 195.3), turned to 0 degrees
- moved D174 2.38 mm to (202.4, 195.3), turned to 0 degrees
- moved D1 1.10 mm to (336.7, 163.9)
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Routing:
- net /Key Matrix/ROW_5: track 0.00 -> 321.9 mm
- net /Key Matrix/ROW_4: track 0.00 -> 262.5 mm
- net Net-(D166-Pad2): track 0.00 -> 37.0 mm
- net Net-(D164-Pad2): track 0.00 -> 30.3 mm
- net Net-(D174-Pad4): track 0.00 -> 30.0 mm
- net Net-(D169-Pad4): track 0.00 -> 28.8 mm
- net Net-(D123-Pad4): track 0.00 -> 26.6 mm
- net Net-(D135-Pad2): track 0.00 -> 24.8 mm
- net /Key Matrix/COL_14: track 48.9 -> 72.7 mm, vias 0 -> 2
- net /Key Matrix/ROW_3: track 250.2 -> 273.1 mm
- net Net-(D153-Pad4): track 0.00 -> 22.9 mm
- net Net-(D178-Pad4): track 0.00 -> 20.9 mm
- net Net-(D140-Pad4): track 0.00 -> 20.8 mm
- net Net-(D167-Pad4): track 0.00 -> 18.4 mm
- net Net-(D177-Pad4): track 0.00 -> 18.4 mm
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