File: mcu.kicad_sch (KiCad schematic)
At the start: 17 parts

Commit message: first draft
Parts:
- removed R?: 0, symbol Device:R
- added J2: Conn_02x03_Odd_Even, symbol Connector_Generic:Conn_02x03_Odd_Even
- added R2, R3, R4: 0R, symbol Device:R
- added R7, R8: 22R, symbol Device:R
- added TP24, TP25: TestPoint, symbol Connector:TestPoint
- gave numbers to parts that had none: 16
Connections:
- net I2C_SCL is gone; now on net ROW_5: U1.18 (PD0)
- net GND: now also J2.6 (Pin_6)
- net ROW_0: now also U1.8 (PB0); no longer U1.1 (PE6)
- net ROW_1: now also U1.9 (PB1), R2.1; no longer U1.8 (PB0)
- net ROW_2: now also U1.10 (PB2), R4.1; no longer U1.9 (PB1)
- net ROW_3: now also U1.11 (PB3), R3.1; no longer U1.10 (PB2)
- net ROW_4: now also U1.12 (PB7); no longer U1.11 (PB3)
- net ROW_5: no longer U1.12 (PB7)
- net VCC: now also J2.2 (Pin_2), TP24.1
- net ~{RST}: now reaches R1.2, SW1.2, U1.13 (~{RESET})
- net ~{RST}: now also J2.5 (Pin_5)
- net D+: no longer names the net of J1.A6 (D+), J1.B6 (D+)
- net D+: now also R8.1; no longer U1.4 (D+)
- net D-: no longer names the net of J1.A7 (D-), J1.B7 (D-)
- net D-: now also R7.2; no longer U1.3 (D-)
- net I2C_SDA: no longer names the net of U1.19 (PD1)
- new net: R8.2, U1.3 (D-)
- new net: R7.1, U1.4 (D+)
- new net LED: U1.1 (PE6)
- new net MISO: J2.1 (Pin_1), R3.2
- new net MOSI: J2.4 (Pin_4), R4.2
- new net SCK: J2.3 (Pin_3), R2.2
- no-connect marks 3 -> 4
Other:
- note removed: "Pull down for both MCU bootstrapping and ISSI LED Driver."
- moved on the sheet: C1, C2, C3, C4, C5, C6, C7, C8, J1, R1, R5, R6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

Commit message: tweaked some bits
Parts:
- added TH1: 500mA, symbol Device:Thermistor_PTC
- X1: value XTAL_GND -> 16MHz
Connections:
- net GND: now also TP25.1
- net VCC: now also TH1.1; no longer J1.A4 (VBUS), J1.A9 (VBUS), J1.B4 (VBUS), J1.B9 (VBUS)
- new net: J1.A4 (VBUS), J1.A9 (VBUS), J1.B4 (VBUS), J1.B9 (VBUS), TH1.2
Other:
- note added: "Place close to MCU"
- moved on the sheet: J1, R5, R6

Commit message: more tweaks
Parts:
- added D1: D, symbol Device:D
- J1: value USB_C_Receptacle_USB2.0 -> USB-C
- J2: value Conn_02x03_Odd_Even -> ISP Header
- R9: value 100k -> 10k
Connections:
- net VCC: now also D1.1 (K)
- net ~{RST}: now also D1.2 (A)
Other:
- note added: "Maybe change value if I decide I want to USB 3.0 only."
- moved on the sheet: R7, R8
Changed lines of the file:
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@@
   (junction (at 162.433 46.101) (diameter 0) (color 0 0 0 0)
   )
+  (junction (at 127 68.961) (diameter 0) (color 0 0 0 0)
+  )
   (junction (at 154.178 39.751) (diameter 0) (color 0 0 0 0)
   )
@@
   )
   (junction (at 87.376 96.901) (diameter 0) (color 0 0 0 0)
+  )
+  (junction (at 123.825 59.182) (diameter 0) (color 0 0 0 0)
   )
   (junction (at 189.484 76.581) (diameter 0) (color 0 0 0 0)
@@
     (stroke (width 0) (type default) (color 0 0 0 0))
   )
+  (wire (pts (xy 127 67.31) (xy 127 68.961))
+    (stroke (width 0) (type default) (color 0 0 0 0))
+  )
   (wire (pts (xy 195.326 85.217) (xy 195.326 87.503))
     (stroke (width 0) (type default) (color 0 0 0 0))
@@
     (stroke (width 0) (type default) (color 0 0 0 0))
   )
+  (wire (pts (xy 127 68.961) (xy 138.938 68.961))
+    (stroke (width 0) (type default) (color 0 0 0 0))
+  )
   (wire (pts (xy 87.376 91.821) (xy 86.741 91.821))
     (stroke (width 0) (type default) (color 0 0 0 0))
@@
     (stroke (width 0) (type default) (color 0 0 0 0))
   )
-  (wire (pts (xy 87.376 96.901) (xy 127.508 96.901))
+  (wire (pts (xy 87.376 96.901) (xy 128.778 96.901))
     (stroke (width 0) (type default) (color 0 0 0 0))
   )
@@
     (stroke (width 0) (type default) (color 0 0 0 0))
   )
+  (wire (pts (xy 123.825 58.166) (xy 123.825 59.182))
+    (stroke (width 0) (type default) (color 0 0 0 0))
+  )
   (wire (pts (xy 189.484 76.581) (xy 189.484 77.597))
     (stroke (width 0) (type default) (color 0 0 0 0))
@@
     (stroke (width 0) (type default) (color 0 0 0 0))
   )
-  (wire (pts (xy 87.376 94.361) (xy 127.508 94.361))
+  (wire (pts (xy 87.376 94.361) (xy 128.778 94.361))
     (stroke (width 0) (type default) (color 0 0 0 0))
   )
@@
     (stroke (width 0) (type default) (color 0 0 0 0))
   )
+  (wire (pts (xy 123.825 59.182) (xy 120.523 59.182))
+    (stroke (width 0) (type default) (color 0 0 0 0))
+  )
   (wire (pts (xy 212.979 95.25) (xy 217.932 95.25))
     (stroke (width 0) (type default) (color 0 0 0 0))
@@
     (stroke (width 0) (type default) (color 0 0 0 0))
   )
+  (wire (pts (xy 120.523 59.182) (xy 120.523 59.436))
+    (stroke (width 0) (type default) (color 0 0 0 0))
+  )
   (wire (pts (xy 169.418 129.921) (xy 170.688 129.921))
     (stroke (width 0) (type default) (color 0 0 0 0))
@@
     (stroke (width 0) (type default) (color 0 0 0 0))
   )
-  (wire (pts (xy 135.128 94.361) (xy 138.938 94.361))
+  (wire (pts (xy 136.398 94.361) (xy 138.938 94.361))
     (stroke (width 0) (type default) (color 0 0 0 0))
   )
@@
     (stroke (width 0) (type default) (color 0 0 0 0))
   )
+  (wire (pts (xy 127 59.69) (xy 127 59.182))
+    (stroke (width 0) (type default) (color 0 0 0 0))
+  )
   (wire (pts (xy 183.642 85.217) (xy 183.642 95.25))
     (stroke (width 0) (type default) (color 0 0 0 0))
@@
     (stroke (width 0) (type default) (color 0 0 0 0))
   )
+  (wire (pts (xy 127 59.182) (xy 123.825 59.182))
+    (stroke (width 0) (type default) (color 0 0 0 0))
+  )
   (wire (pts (xy 169.418 112.141) (xy 170.688 112.141))
     (stroke (width 0) (type default) (color 0 0 0 0))
@@
     (stroke (width 0) (type default) (color 0 0 0 0))
   )
-  (wire (pts (xy 120.523 58.166) (xy 120.523 59.436))
-    (stroke (width 0) (type default) (color 0 0 0 0))
-  )
   (wire (pts (xy 156.718 61.341) (xy 156.718 60.706))
     (stroke (width 0) (type default) (color 0 0 0 0))
@@
     (stroke (width 0) (type default) (color 0 0 0 0))
   )
-  (wire (pts (xy 135.128 96.901) (xy 138.938 96.901))
+  (wire (pts (xy 136.398 96.901) (xy 138.938 96.901))
     (stroke (width 0) (type default) (color 0 0 0 0))
   )
@@
     (stroke (width 0) (type default) (color 0 0 0 0))
   )
-  (wire (pts (xy 120.523 68.961) (xy 138.938 68.961))
+  (wire (pts (xy 120.523 68.961) (xy 127 68.961))
     (stroke (width 0) (type default) (color 0 0 0 0))
   )
@@
   (wire (pts (xy 120.523 67.056) (xy 120.523 68.961))
     (stroke (width 0) (type default) (color 0 0 0 0))
+  )
+  (text "Maybe change value \nif I decide I want \nto USB 3.0 only."
+    (at 67.31 68.961 0)
+    (effects (font (size 1.27 1.27)) (justify left bottom))
   )
   (text "Place close to MCU" (at 164.084 38.735 180)
@@
     (pin "2")
   )
-  (symbol (lib_id "Device:R") (at 131.318 94.361 270) (unit 1)
-    (in_bom yes) (on_board yes)
-    (property "Reference" "R7" (id 0) (at 131.318 94.361 90))
-    (property "Value" "22R" (id 1) (at 131.318 91.821 90))
-    (property "Footprint" "" (id 2) (at 131.318 92.583 90)
-      (effects (font (size 1.27 1.27)) hide)
-    )
-    (property "Datasheet" "~" (id 3) (at 131.318 94.361 0)
+  (symbol (lib_id "Device:R") (at 132.588 94.361 270) (unit 1)
+    (in_bom yes) (on_board yes)
+    (property "Reference" "R7" (id 0) (at 132.588 94.361 90))
+    (property "Value" "22R" (id 1) (at 132.588 91.821 90))
+    (property "Footprint" "" (id 2) (at 132.588 92.583 90)
+      (effects (font (size 1.27 1.27)) hide)
+    )
+    (property "Datasheet" "~" (id 3) (at 132.588 94.361 0)
       (effects (font (size 1.27 1.27)) hide)
     )
@@
     (pin "1")
   )
-  (symbol (lib_id "power:VCC") (at 120.523 58.166 0) (unit 1)
-    (in_bom yes) (on_board yes) (fields_autoplaced)
-    (property "Reference" "#PWR05" (id 0) (at 120.523 61.976 0)
-      (effects (font (size 1.27 1.27)) hide)
-    )
-    (property "Value" "VCC" (id 1) (at 120.523 54.5902 0))
-    (property "Footprint" "" (id 2) (at 120.523 58.166 0)
-      (effects (font (size 1.27 1.27)) hide)
-    )
-    (property "Datasheet" "" (id 3) (at 120.523 58.166 0)
+  (symbol (lib_id "power:VCC") (at 123.825 58.166 0) (unit 1)
+    (in_bom yes) (on_board yes) (fields_autoplaced)
+    (property "Reference" "#PWR05" (id 0) (at 123.825 61.976 0)
+      (effects (font (size 1.27 1.27)) hide)
+    )
+    (property "Value" "VCC" (id 1) (at 123.825 54.5902 0))
+    (property "Footprint" "" (id 2) (at 123.825 58.166 0)
+      (effects (font (size 1.27 1.27)) hide)
+    )
+    (property "Datasheet" "" (id 3) (at 123.825 58.166 0)
       (effects (font (size 1.27 1.27)) hide)
     )
@@
     (in_bom yes) (on_board yes) (fields_autoplaced)
     (property "Reference" "J1" (id 0) (at 71.501 72.8812 0))
-    (property "Value" "USB_C_Receptacle_USB2.0" (id 1) (at 71.501 75.4181 0))
+    (property "Value" "USB-C" (id 1) (at 71.501 75.4181 0))
     (property "Footprint" "" (id 2) (at 75.311 94.361 0)
       (effects (font (size 1.27 1.27)) hide)
@@
       (effects (font (size 1.27 1.27)) (justify left))
     )
-    (property "Value" "100k" (id 1) (at 183.896 128.6479 0)
+    (property "Value" "10k" (id 1) (at 183.896 128.6479 0)
       (effects (font (size 1.27 1.27)) (justify left))
     )
@@
     (in_bom yes) (on_board yes)
     (property "Reference" "J2" (id 0) (at 206.502 90.297 0))
-    (property "Value" "Conn_02x03_Odd_Even" (id 1) (at 200.152 101.092 0)
-      (effects (font (size 1.27 1.27)) hide)
-    )
+    (property "Value" "ISP Header" (id 1) (at 206.629 100.203 0))
     (property "Footprint" "" (id 2) (at 205.359 95.25 0)
       (effects (font (size 1.27 1.27)) hide)
@@
     (pin "2")
   )
+  (symbol (lib_id "Device:D") (at 127 63.5 270) (unit 1)
+    (in_bom yes) (on_board yes)
+    (property "Reference" "D1" (id 0) (at 128.397 63.5 90)
+      (effects (font (size 1.27 1.27)) (justify left))
+    )
+    (property "Value" "D" (id 1) (at 128.524 64.516 90)
+      (effects (font (size 1.27 1.27)) (justify left) hide)
+    )
+    (property "Footprint" "" (id 2) (at 127 63.5 0)
+      (effects (font (size 1.27 1.27)) hide)
+    )
+    (property "Datasheet" "~" (id 3) (at 127 63.5 0)
+      (effects (font (size 1.27 1.27)) hide)
+    )
+    (pin "1")
+    (pin "2")
+  )
   (symbol (lib_id "power:PWR_FLAG") (at 157.988 24.257 180) (unit 1)
     (in_bom yes) (on_board yes) (fields_autoplaced)
@@
     (pin "1")
   )
-  (symbol (lib_id "Device:R") (at 131.318 96.901 90) (unit 1)
-    (in_bom yes) (on_board yes)
-    (property "Reference" "R8" (id 0) (at 131.318 96.901 90))
-    (property "Value" "22R" (id 1) (at 131.318 99.441 90))
-    (property "Footprint" "" (id 2) (at 131.318 98.679 90)
-      (effects (font (size 1.27 1.27)) hide)
-    )
-    (property "Datasheet" "~" (id 3) (at 131.318 96.901 0)
-      (effects (font (size 1.27 1.27)) hide)
-    )
+  (symbol (lib_id "Device:R") (at 132.588 96.901 90) (unit 1)
+    (in_bom yes) (on_board yes)
+    (property "Reference" "R8" (id 0) (at 132.588 96.901 90))
+    (property "Value" "22R" (id 1) (at 132.588 99.441 90))
+    (property "Footprint" "" (id 2) (at 132.588 98.679 90)
+      (effects (font (size 1.27 1.27)) hide)
+    )
+    (property "Datasheet" "~" (id 3) (at 132.588 96.901 0)
+      (effects (font (size 1.27 1.27)) hide)
+    )

Commit message: keyswitch placement
Parts:
- removed X1: 16MHz, symbol tmk-sym:XTAL_GND
- added Y1: 16MHz, Custom:Crystal_SMD_3225-4Pin_3.2x2.5mm_HandSoldering, symbol Device:Crystal_GND2_Small
- C1, C2, C3, C4, C5, C6, C7, C8: footprint (none) -> Capacitor_SMD:C_0805_2012Metric_Pad1.18x1.45mm_HandSolder
- D1: value D -> 1N4148; footprint (none) -> Diode_SMD:D_SOD-123
- J1: footprint (none) -> Connector_USB:USB_C_Receptacle_XKB_U262-16XN-4BVC11
- J2: footprint (none) -> Connector_PinHeader_2.54mm:PinHeader_2x03_P2.54mm_Vertical
- R1, R2, R3, R4, R5, R6, R7, R8, R9: footprint (none) -> Resistor_SMD:R_0805_2012Metric_Pad1.20x1.40mm_HandSolder
- SW1: footprint (none) -> Button_Switch_SMD:SW_Push_1P1T_NO_6x6mm_H9.5mm
- TH1: value 500mA -> 500mA PTC; footprint (none) -> Resistor_SMD:R_1206_3216Metric_Pad1.30x1.75mm_HandSolder
- TP24, TP25: footprint (none) -> TestPoint:TestPoint_THTPad_D1.0mm_Drill0.5mm
Connections:
- net GND: now also Y1.2
- net at C7.1, U1.16 (XTAL2): now also Y1.3
- net at C6.1, U1.17 (XTAL1): now also Y1.1

Commit message: more layout
Parts:
- renumbered J2 to J1, J1 to J2, R7 to R5, R5 to R6, R8 to R7, R6 to R8
Connections:
- net XTAL2: now reaches C7.1, U1.16 (XTAL2), Y1.3
- net XTAL1: now reaches C6.1, U1.17 (XTAL1), Y1.1
- net MCU_D-: now reaches R7.2, U1.3 (D-)
- net ~{HWB}: now reaches R9.1, U1.33 (~{HWB}/PE2)
- net MCU_D+: now reaches R5.1, U1.4 (D+)
- net UCAP: now reaches C8.1, U1.6 (UCAP)
- net CON_D-: now reaches J2.A7 (D-), J2.B7 (D-)
- net CON_D-: now also R7.1; no longer R5.2
- net VBUS: now reaches J2.A4 (VBUS), J2.A9 (VBUS), J2.B4 (VBUS), J2.B9 (VBUS), TH1.2
- net CC1: now reaches J2.A5 (CC1), R6.2
- net CON_D+: now reaches J2.A6 (D+), J2.B6 (D+)
- net CON_D+: now also R5.2; no longer R7.1
- net CC2: now reaches J2.B5 (CC2), R8.1
Other:
- moved on the sheet: J2, R5, R6, R7, R8, TH1
