File: LEDS.kicad_sch (KiCad schematic)
At the start: 12 parts

Commit message: first draft
Parts:
- removed C? (x4): 0.1u, symbol Device:C_Small
- removed C? (x3): 1u, symbol Device:C_Small
- removed R?: 10k, symbol Device:R
- removed R? (x2): 2k, symbol Device:R
- removed U? (x2): IS31FL3741A, symbol Custom:IS31FL3741A
- added D100, D101, D102, D103, D104, D105, D106, D107, D108, D109, D110, D111, D112, D113, D114, D115, D116, D117, D118, D119, D120, D121, D122, D123, D124, D125, D126, D127, D128, D129, D130, D131, D132, D133, D134, D135, D136, D137, D138, D139, D140, D141, D142, D143, D144, D145, D146, D147, D148, D149, D150, D151, D152, D153, D154, D155, D156, D157, D158, D159, D160, D161, D162, D163, D164, D165, D166, D167, D168, D169, D170, D171, D172, D173, D174, D175, D176, D177, D178, D179, D180, D89, D90, D91, D92, D93, D94, D95, D96, D97, D98, D99: SK6803MINI-E, symbol Custom:SK6803MINI-E
- added J3: Conn_01x03, symbol Connector_Generic:Conn_01x03
Connections:
- net GND: now also D100.1 (GND), D101.1 (GND), D102.1 (GND), D103.1 (GND), D104.1 (GND), D105.1 (GND), D106.1 (GND), D107.1 (GND), D108.1 (GND), D109.1 (GND), D110.1 (GND), D111.1 (GND), D112.1 (GND), D113.1 (GND), D114.1 (GND), D115.1 (GND), D116.1 (GND), D117.1 (GND), D118.1 (GND), D119.1 (GND), D120.1 (GND), D121.1 (GND), D122.1 (GND), D123.1 (GND), D124.1 (GND), D125.1 (GND), D126.1 (GND), D127.1 (GND), D128.1 (GND), D129.1 (GND), D130.1 (GND), D131.1 (GND), D132.1 (GND), D133.1 (GND), D134.1 (GND), D135.1 (GND), D136.1 (GND), D137.1 (GND), D138.1 (GND), D139.1 (GND), D140.1 (GND), D141.1 (GND), D142.1 (GND), D143.1 (GND), D144.1 (GND), D145.1 (GND), D146.1 (GND), D147.1 (GND), D148.1 (GND), D149.1 (GND), D150.1 (GND), D151.1 (GND), D152.1 (GND), D153.1 (GND), D154.1 (GND), D155.1 (GND), D156.1 (GND), D157.1 (GND), D158.1 (GND), D159.1 (GND), D160.1 (GND), D161.1 (GND), D162.1 (GND), D163.1 (GND), D164.1 (GND), D165.1 (GND), D166.1 (GND), D167.1 (GND), D168.1 (GND), D169.1 (GND), D170.1 (GND), D171.1 (GND), D172.1 (GND), D173.1 (GND), D174.1 (GND), D175.1 (GND), D176.1 (GND), D177.1 (GND), D178.1 (GND), D179.1 (GND), D180.1 (GND), D89.1 (GND), D90.1 (GND), D91.1 (GND), D92.1 (GND), D93.1 (GND), D94.1 (GND), D95.1 (GND), D96.1 (GND), D97.1 (GND), D98.1 (GND), D99.1 (GND), J3.2 (Pin_2)
- net VCC: now also D100.3 (VDD), D101.3 (VDD), D102.3 (VDD), D103.3 (VDD), D104.3 (VDD), D105.3 (VDD), D106.3 (VDD), D107.3 (VDD), D108.3 (VDD), D109.3 (VDD), D110.3 (VDD), D111.3 (VDD), D112.3 (VDD), D113.3 (VDD), D114.3 (VDD), D115.3 (VDD), D116.3 (VDD), D117.3 (VDD), D118.3 (VDD), D119.3 (VDD), D120.3 (VDD), D121.3 (VDD), D122.3 (VDD), D123.3 (VDD), D124.3 (VDD), D125.3 (VDD), D126.3 (VDD), D127.3 (VDD), D128.3 (VDD), D129.3 (VDD), D130.3 (VDD), D131.3 (VDD), D132.3 (VDD), D133.3 (VDD), D134.3 (VDD), D135.3 (VDD), D136.3 (VDD), D137.3 (VDD), D138.3 (VDD), D139.3 (VDD), D140.3 (VDD), D141.3 (VDD), D142.3 (VDD), D143.3 (VDD), D144.3 (VDD), D145.3 (VDD), D146.3 (VDD), D147.3 (VDD), D148.3 (VDD), D149.3 (VDD), D150.3 (VDD), D151.3 (VDD), D152.3 (VDD), D153.3 (VDD), D154.3 (VDD), D155.3 (VDD), D156.3 (VDD), D157.3 (VDD), D158.3 (VDD), D159.3 (VDD), D160.3 (VDD), D161.3 (VDD), D162.3 (VDD), D163.3 (VDD), D164.3 (VDD), D165.3 (VDD), D166.3 (VDD), D167.3 (VDD), D168.3 (VDD), D169.3 (VDD), D170.3 (VDD), D171.3 (VDD), D172.3 (VDD), D173.3 (VDD), D174.3 (VDD), D175.3 (VDD), D176.3 (VDD), D177.3 (VDD), D178.3 (VDD), D179.3 (VDD), D180.3 (VDD), D89.3 (VDD), D90.3 (VDD), D91.3 (VDD), D92.3 (VDD), D93.3 (VDD), D94.3 (VDD), D95.3 (VDD), D96.3 (VDD), D97.3 (VDD), D98.3 (VDD), D99.3 (VDD), J3.1 (Pin_1)
- new net: D141.4 (DOUT), D142.2 (DIN)
- new net: D142.4 (DOUT), D143.2 (DIN)
- new net: D148.4 (DOUT), D149.2 (DIN)
- new net: D149.4 (DOUT), D150.2 (DIN)
- new net: D134.2 (DIN), D135.4 (DOUT)
- new net: D133.2 (DIN), D134.4 (DOUT)
- new net: D105.4 (DOUT), D106.2 (DIN)
- new net: D106.4 (DOUT), D107.2 (DIN)
- new net: D130.2 (DIN), D131.4 (DOUT)
- new net: D129.2 (DIN), D130.4 (DOUT)
- new net: D100.2 (DIN), D101.4 (DOUT)
- new net: D100.4 (DOUT), D99.2 (DIN)
- new net: D126.2 (DIN), D127.4 (DOUT)
- new net: D125.2 (DIN), D126.4 (DOUT)
- new net: D165.2 (DIN), D180.4 (DOUT)
- new net: D165.4 (DOUT), J3.3 (Pin_3)
- new net: D97.2 (DIN), D98.4 (DOUT)
- new net: D96.2 (DIN), D97.4 (DOUT)
- new net: D109.4 (DOUT), D110.2 (DIN)
- new net: D110.4 (DOUT), D111.2 (DIN)
- new net: D147.4 (DOUT), D148.2 (DIN)
- new net: D146.4 (DOUT), D147.2 (DIN)
- new net: D123.2 (DIN), D124.4 (DOUT)
- new net: D122.2 (DIN), D123.4 (DOUT)
- new net: D122.4 (DOUT), D139.2 (DIN)
- new net: D171.4 (DOUT), D172.2 (DIN)
- new net: D172.4 (DOUT), D173.2 (DIN)
- new net: D94.2 (DIN), D95.4 (DOUT)
- new net: D93.2 (DIN), D94.4 (DOUT)
- new net: D101.2 (DIN), D102.4 (DOUT)
- new net: D105.2 (DIN), D89.4 (DOUT)
- new net: D90.2 (DIN), D91.4 (DOUT)
- new net: D89.2 (DIN), D90.4 (DOUT)
- new net: D95.2 (DIN), D96.4 (DOUT)
- new net: D174.4 (DOUT), D175.2 (DIN)
- new net: D175.4 (DOUT), D176.2 (DIN)
- new net: D116.4 (DOUT), D117.2 (DIN)
- new net: D117.4 (DOUT), D118.2 (DIN)
- new net: D161.2 (DIN), D162.4 (DOUT)
- new net: D160.2 (DIN), D161.4 (DOUT)
- new net: D145.4 (DOUT), D146.2 (DIN)
- new net: D158.2 (DIN), D159.4 (DOUT)
- new net: D157.2 (DIN), D158.4 (DOUT)
- new net: D170.4 (DOUT), D171.2 (DIN)
- new net: D121.4 (DOUT), D138.2 (DIN)
- new net: D137.2 (DIN), D138.4 (DOUT)
- new net: D118.4 (DOUT), D119.2 (DIN)
- new net: D124.2 (DIN), D125.4 (DOUT)
- new net: D152.4 (DOUT), D166.2 (DIN)
- new net: D166.4 (DOUT), D167.2 (DIN)
- new net: D169.4 (DOUT), D170.2 (DIN)
- new net: D152.2 (DIN), D153.4 (DOUT)
- new net: D173.4 (DOUT), D174.2 (DIN)
- new net: D102.2 (DIN), D103.4 (DOUT)
- new net: D92.2 (DIN), D93.4 (DOUT)
- new net: D140.4 (DOUT), D141.2 (DIN)
- new net: D132.2 (DIN), D133.4 (DOUT)
- new net: D131.2 (DIN), D132.4 (DOUT)
- new net: D167.4 (DOUT), D168.2 (DIN)
- new net: D168.4 (DOUT), D169.2 (DIN)
- new net: D153.2 (DIN), D154.4 (DOUT)
- new net: D135.2 (DIN), D136.4 (DOUT)
- new net: D150.4 (DOUT), D151.2 (DIN)
- new net: D139.4 (DOUT), D140.2 (DIN)
- new net: D103.2 (DIN), D104.4 (DOUT)
- new net: D159.2 (DIN), D160.4 (DOUT)
- new net: D154.2 (DIN), D155.4 (DOUT)
- new net: D143.4 (DOUT), D144.2 (DIN)
- new net: D112.4 (DOUT), D113.2 (DIN)
- new net: D113.4 (DOUT), D114.2 (DIN)
- new net: D176.4 (DOUT), D177.2 (DIN)
- new net: D120.4 (DOUT), D121.2 (DIN)
- new net: D111.4 (DOUT), D112.2 (DIN)
- new net: D108.4 (DOUT), D109.2 (DIN)
- new net: D128.2 (DIN), D129.4 (DOUT)
- new net: D107.4 (DOUT), D108.2 (DIN)
- new net: D162.2 (DIN), D163.4 (DOUT)
- new net: D119.4 (DOUT), D120.2 (DIN)
- new net: D177.4 (DOUT), D178.2 (DIN)
- new net: D178.4 (DOUT), D179.2 (DIN)
- new net: D115.4 (DOUT), D116.2 (DIN)
- new net: D114.4 (DOUT), D115.2 (DIN)
- new net: D156.2 (DIN), D157.4 (DOUT)
- new net: D127.2 (DIN), D128.4 (DOUT)
- new net: D151.4 (DOUT), D164.2 (DIN)
- new net: D144.4 (DOUT), D145.2 (DIN)
- new net: D91.2 (DIN), D92.4 (DOUT)
- new net: D155.2 (DIN), D156.4 (DOUT)
- new net: D98.2 (DIN), D99.4 (DOUT)
- new net: D136.2 (DIN), D137.4 (DOUT)
- new net: D163.2 (DIN), D164.4 (DOUT)
- new net: D179.4 (DOUT), D180.2 (DIN)
- new net LEDs: D104.2 (DIN)
- no-connect marks 1 -> 0

Commit message: tweaked some bits
Parts:
- added R10: 470R, symbol Device:R
Connections:
- net LEDs: now also R10.2; no longer D104.2 (DIN)
- new net: D104.2 (DIN), R10.1
Other:
- note added: "Note: all of these running with all channels at full brightness would draw 920mA, which blows right past the USB 2.0 and 3.0 spec. Fortunately for us, on full brightness they are very fucking bright, and so we can easily get away with probably 20% power (which, thanks to Weber's law, is only about half the perceived brightness!). That would lose us a good bit of dynamic range though. It's somethi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"
Changed lines of the file:
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@@
-    (stroke (width 0) (type default) (color 0 0 0 0))
-  )
-  (wire (pts (xy 281.686 31.75) (xy 282.448 31.75))
     (stroke (width 0) (type default) (color 0 0 0 0))
   )
@@
     (stroke (width 0) (type default) (color 0 0 0 0))
   )
+  (wire (pts (xy 281.94 31.75) (xy 281.686 31.75))
+    (stroke (width 0) (type default) (color 0 0 0 0))
+  )
   (wire (pts (xy 84.963 155.448) (xy 84.963 155.702))
     (stroke (width 0) (type default) (color 0 0 0 0))
@@
     (stroke (width 0) (type default) (color 0 0 0 0))
   )
+  (wire (pts (xy 268.859 16.51) (xy 270.256 16.51))
+    (stroke (width 0) (type default) (color 0 0 0 0))
+  )
   (wire (pts (xy 234.442 78.232) (xy 234.95 78.232))
     (stroke (width 0) (type default) (color 0 0 0 0))
@@
     (stroke (width 0) (type default) (color 0 0 0 0))
   )
-  (wire (pts (xy 282.448 30.226) (xy 282.448 31.75))
-    (stroke (width 0) (type default) (color 0 0 0 0))
-  )
   (wire (pts (xy 100.838 116.84) (xy 100.838 117.094))
     (stroke (width 0) (type default) (color 0 0 0 0))
@@
     (stroke (width 0) (type default) (color 0 0 0 0))
   )
+  (wire (pts (xy 277.876 16.51) (xy 281.94 16.51))
+    (stroke (width 0) (type default) (color 0 0 0 0))
+  )
   (wire (pts (xy 37.846 47.117) (xy 37.846 47.371))
     (stroke (width 0) (type default) (color 0 0 0 0))
@@
     (stroke (width 0) (type default) (color 0 0 0 0))
   )
+  (wire (pts (xy 281.94 16.51) (xy 281.94 31.75))
+    (stroke (width 0) (type default) (color 0 0 0 0))
+  )
   (wire (pts (xy 53.594 109.093) (xy 53.594 109.347))
     (stroke (width 0) (type default) (color 0 0 0 0))
@@
     (stroke (width 0) (type default) (color 0 0 0 0))
   )
-  (hierarchical_label "LEDs" (shape input) (at 282.448 30.226 90)
-    (effects (font (size 1.27 1.27)) (justify left))
+  (text "Note: all of these running with all channels at full \nbrightness would draw 920mA, which blows right past\nthe USB 2.0 and 3.0 spec. Fortunately for us, on \nfull brightness they are very fucking bright, and\nso we can easily get away with probably 20% power\n(which, thanks to Weber's law, is only about half the\nperceived brightness!). That would lose us a good bit\nof dynamic range though. It's something to play with."
+    (at 16.891 193.548 0)
+    (effects (font (size 2.54 2.54)) (justify left bottom))
+  )
+  (hierarchical_label "LEDs" (shape input) (at 268.859 16.51 180)
+    (effects (font (size 1.27 1.27)) (justify right))
   )
   (symbol (lib_id "power:VCC") (at 258.191 139.954 0) (unit 1)
@@
     (pin "1")
   )
+  (symbol (lib_id "Device:R") (at 274.066 16.51 270) (unit 1)
+    (in_bom yes) (on_board yes)
+    (property "Reference" "R10" (id 0) (at 272.161 14.478 90)
+      (effects (font (size 1.27 1.27)) (justify left))
+    )
+    (property "Value" "470R" (id 1) (at 271.78 18.796 90)
+      (effects (font (size 1.27 1.27)) (justify left))
+    )
+    (property "Footprint" "" (id 2) (at 274.066 14.732 90)
+      (effects (font (size 1.27 1.27)) hide)
+    )
+    (property "Datasheet" "~" (id 3) (at 274.066 16.51 0)
+      (effects (font (size 1.27 1.27)) hide)
+    )
+    (pin "1")
+    (pin "2")
+  )
   (symbol (lib_id "power:GND") (at 53.467 155.702 0) (unit 1)

Commit message: more tweaks
Parts:
- J3: value Conn_01x03 -> LED Extension
- renumbered D99 to D100, D100 to D101, D101 to D102, D102 to D103, D103 to D104, D104 to D105, D105 to D106, D106 to D107, D107 to D108, D108 to D109, D109 to D110, D110 to D111, D111 to D112, D112 to D113, D113 to D114, D114 to D115, D115 to D116, D116 to D117, D117 to D118, D118 to D119, D119 to D120, D120 to D121, D121 to D122, D122 to D123, D123 to D124, D124 to D125, D125 to D126, D126 to D127, D127 to D128, D128 to D129, D129 to D130, D130 to D131, D131 to D132, D132 to D133, D133 to D134, D134 to D135, D135 to D136, D136 to D137, D137 to D138, D138 to D139, D139 to D140, D140 to D141, D141 to D142, D142 to D143, D143 to D144, D144 to D145, D145 to D146, D146 to D147, D147 to D148, D148 to D149, D149 to D150, D150 to D151, D151 to D152, D152 to D153, D153 to D154, D154 to D155, D155 to D156, D156 to D157, D157 to D158, D158 to D159, D159 to D160, D160 to D161, D161 to D162, D162 to D163, D163 to D164, D164 to D165, D165 to D166, D166 to D167, D167 to D168, D168 to D169, D169 to D170, D170 to D171, D171 to D172, D172 to D173, D173 to D174, D174 to D175, D175 to D176, D176 to D177, D177 to D178, D178 to D179, D179 to D180, D180 to D181, D89 to D90, D90 to D91, D91 to D92, D92 to D93, D93 to D94, D94 to D95, D95 to D96, D96 to D97, D97 to D98, D98 to D99
Connections:
- net LEDs renamed LED

Commit message: keyswitch placement
Parts:
- D100, D101, D102, D103, D104, D105, D106, D107, D108, D109, D110, D111, D112, D113, D114, D115, D116, D117, D118, D119, D120, D121, D122, D123, D124, D125, D126, D127, D128, D129, D130, D131, D132, D133, D134, D135, D136, D137, D138, D139, D140, D141, D142, D143, D144, D145, D146, D147, D148, D149, D150, D151, D152, D153, D154, D155, D156, D157, D158, D159, D160, D161, D162, D163, D164, D165, D166, D167, D168, D169, D170, D171, D172, D173, D174, D175, D176, D177, D178, D179, D180, D181, D90, D91, D92, D93, D94, D95, D96, D97, D98, D99: footprint (none) -> Custom:SK6803MINI-E_Bottom_Up
- J3: footprint (none) -> Connector_PinHeader_2.54mm:PinHeader_1x03_P2.54mm_Horizontal
- R10: footprint (none) -> Resistor_SMD:R_0805_2012Metric_Pad1.20x1.40mm_HandSolder

Commit message: rough layout complete
Parts:
- R10: footprint Resistor_SMD:R_0805_2012Metric_Pad1.20x1.40mm_HandSolder -> Resistor_SMD:R_0603_1608Metric_Pad0.98x0.95mm_HandSolder
Changed lines of the file:
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@@
       (effects (font (size 1.27 1.27)) (justify left))
     )
-    (property "Footprint" "Resistor_SMD:R_0805_2012Metric_Pad1.20x1.40mm_HandSolder" (id 2) (at 274.066 14.732 90)
+    (property "Footprint" "Resistor_SMD:R_0603_1608Metric_Pad0.98x0.95mm_HandSolder" (id 2) (at 274.066 14.732 90)
       (effects (font (size 1.27 1.27)) hide)
     )

Commit message: needs lots of tidying
Parts:
- added C10, C100, C11, C12, C13, C14, C15, C16, C17, C18, C19, C20, C21, C22, C23, C24, C25, C26, C27, C28, C29, C30, C31, C32, C33, C34, C35, C36, C37, C38, C39, C40, C41, C42, C43, C44, C45, C46, C47, C48, C49, C50, C51, C52, C53, C54, C55, C56, C57, C58, C59, C60, C61, C62, C63, C64, C65, C66, C67, C68, C69, C70, C71, C72, C73, C74, C75, C76, C77, C78, C79, C80, C81, C82, C83, C84, C85, C86, C87, C88, C89, C9, C90, C91, C92, C93, C94, C95, C96, C97, C98, C99: 100n, Capacitor_SMD:C_0805_2012Metric_Pad1.18x1.45mm_HandSolder, symbol Device:C
Connections:
- net GND: now also C10.2, C100.2, C11.2, C12.2, C13.2, C14.2, C15.2, C16.2, C17.2, C18.2, C19.2, C20.2, C21.2, C22.2, C23.2, C24.2, C25.2, C26.2, C27.2, C28.2, C29.2, C30.2, C31.2, C32.2, C33.2, C34.2, C35.2, C36.2, C37.2, C38.2, C39.2, C40.2, C41.2, C42.2, C43.2, C44.2, C45.2, C46.2, C47.2, C48.2, C49.2, C50.2, C51.2, C52.2, C53.2, C54.2, C55.2, C56.2, C57.2, C58.2, C59.2, C60.2, C61.2, C62.2, C63.2, C64.2, C65.2, C66.2, C67.2, C68.2, C69.2, C70.2, C71.2, C72.2, C73.2, C74.2, C75.2, C76.2, C77.2, C78.2, C79.2, C80.2, C81.2, C82.2, C83.2, C84.2, C85.2, C86.2, C87.2, C88.2, C89.2, C9.2, C90.2, C91.2, C92.2, C93.2, C94.2, C95.2, C96.2, C97.2, C98.2, C99.2
- net LED: now also R10.1; no longer R10.2
- net VCC: now also C10.1, C100.1, C11.1, C12.1, C13.1, C14.1, C15.1, C16.1, C17.1, C18.1, C19.1, C20.1, C21.1, C22.1, C23.1, C24.1, C25.1, C26.1, C27.1, C28.1, C29.1, C30.1, C31.1, C32.1, C33.1, C34.1, C35.1, C36.1, C37.1, C38.1, C39.1, C40.1, C41.1, C42.1, C43.1, C44.1, C45.1, C46.1, C47.1, C48.1, C49.1, C50.1, C51.1, C52.1, C53.1, C54.1, C55.1, C56.1, C57.1, C58.1, C59.1, C60.1, C61.1, C62.1, C63.1, C64.1, C65.1, C66.1, C67.1, C68.1, C69.1, C70.1, C71.1, C72.1, C73.1, C74.1, C75.1, C76.1, C77.1, C78.1, C79.1, C80.1, C81.1, C82.1, C83.1, C84.1, C85.1, C86.1, C87.1, C88.1, C89.1, C9.1, C90.1, C91.1, C92.1, C93.1, C94.1, C95.1, C96.1, C97.1, C98.1, C99.1
- net at D139.2 (DIN): now also R10.2; no longer D122.4 (DOUT)
- net at D119.4 (DOUT): now also D136.2 (DIN); no longer D120.2 (DIN)
- net at D105.2 (DIN): now also D122.4 (DOUT); no longer R10.1
- net at D137.4 (DOUT): now also D120.2 (DIN); no longer D136.2 (DIN)
Other:
- moved on the sheet: D100, D101, D102, D103, D104, D105, D106, D107, D108, D109, D110, D111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
